File: pcb/MusicPad.kicad_pcb (KiCad board)
At the start: 2 copper layers, 65.1 x 65.1 mm, 15 parts, among them J1 OLED_128x32, SW1 SW_Push, SW2 SW_Push, SW3 SW_Push, SW4 SW_Push, SW5 SW_Push, SW6 RotaryEncoder_Switch, U1 XIAO-RP2040-DIP

Commit message: added production files
Other:
- board text added: "XIAO HERE"
Changed lines of the file:
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@@
 			(outputformat 1)
 			(mirror no)
-			(drillshape 1)
+			(drillshape 0)
 			(scaleselection 1)
-			(outputdirectory "")
+			(outputdirectory "../production/")
 		)
 	)
@@
 			)
 			(justify left bottom)
+		)
+	)
+	(gr_text "XIAO HERE"
+		(at 166.6875 66.675 270)
+		(layer "F.SilkS")
+		(effects
+			(font
+				(size 1 1)
+				(thickness 0.1)
+			)
+			(justify left bottom)
